Commit message: feat: 增加新的显示

File: public/sample.urdf (robot description, URDF)
Before this commit: robot simple_robot, 3 links, 2 joints
Links:
- link arm_link_1: geometry collision cylinder length=0.8 radius=0.08; visual cylinder length=0.8 radius=0.08
- link arm_link_2: geometry collision cylinder length=0.6 radius=0.06; visual cylinder length=0.6 radius=0.06
- link base_link: geometry collision box size=0.6 0.6 0.2; visual box size=0.6 0.6 0.2
