Commit message: remove some samples

File: public/1.urdf (robot description, URDF)
Before this commit: robot two_link_arm, 3 links, 2 joints
Links:
- removed link link1
- removed link link2
- added link arm_link_1; collision cylinder length=0.8 radius=0.08; visual cylinder length=0.8 radius=0.08
- added link arm_link_2; collision cylinder length=0.6 radius=0.06; visual cylinder length=0.6 radius=0.06
- link base_link: geometry collision box size=0.6 0.6 0.2; visual box size=0.6 0.6 0.2
Joints:
- removed joint elbow_joint
- removed joint shoulder_joint
- added joint arm_1_to_arm_2: type revolute, parent arm_link_1, child arm_link_2, origin xyz=0 0 0.8 rpy=0 1.5707 0, axis 0 1 0, limit lower=-1.5707 upper=1.5707 effort=100 velocity=100
- added joint base_to_arm_1: type revolute, parent base_link, child arm_link_1, origin xyz=0 0 0.1 rpy=0 0 0, axis 0 0 1, limit lower=-3.1415 upper=3.1415 effort=100 velocity=100
